File: schematic.sch (EAGLE design)
At the start: 365 parts, among them CON1 UBC05V128-B0C04D, IC1 FT232RL, IC10 TL084D, IC13 7805TV, IC3 TL084D, IC4 TL084D, IC5 TL084D, IC6 TL084D, IC7 TL084D, IC8 TL084D, IC9 TL084D, Q2 BC557, T1 BC547, T2 BC547, U1 TMS320F28069_PN_80, U2 TLV5610_PW_20, U3 REF2030AIDDCR, U5 TS12A44514DR, U6 TS12A44514DR, U7 TPS7333QD, U9 MAX395CWG+

Commit message: modified limiting circuit
Parts:
- removed R106, R126, R128, R130, R132, R134, R136, R138: (no value), rcl:R-US_R1206
- JP28: value (none) -> Useless
- JP34: value (none) -> pls
- JP41: value (none) -> adc_in
- JP44: value (none) -> Int_inp
Connections:
- net +1.5V: now also C54.1, C55.1, C56.1, C57.1, C58.1, C59.1, C60.1, C61.1, R100.1, R104.1, R41.1, R58.1, R62.1, R66.1, R70.1, R82.1
- net +3V3: no longer R125.2, R127.2, R129.2, R131.2, R133.2, R135.2, R137.2, R14.2
- net +5V: no longer C54.1, C55.1, C56.1, C57.1, C58.1, C59.1, C60.1, C61.1, R100.1, R104.1, R41.1, R58.1, R62.1, R66.1, R70.1, R82.1
- net AGND: no longer R106.1, R126.1, R128.1, R130.1, R132.1, R134.1, R136.1, R138.1
- net N$118: now also R14.2; no longer R106.2
- net N$119: now also R125.2; no longer R126.2
- net N$120: now also R127.2; no longer R128.2
- net N$122: now also R129.2; no longer R130.2
- net N$124: now also R131.2; no longer R132.2
- net N$126: now also R133.2; no longer R134.2
- net N$128: now also R135.2; no longer R136.2
- net N$130: now also R137.2; no longer R138.2
