File: March 9/schematic_March8.brd (EAGLE design)
At the start: 215.6 x 361.3 mm, 314 parts, among them CON1 UBC05V128-B0C04D, IC1 FT232RL, IC10 TL084D, IC13 7805TV, IC3 TL084D, IC4 TL084D, IC5 TL084D, IC6 TL084D, IC7 TL084D, IC8 TL084D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

Commit message: Began digital part ka routing
Parts:
- moved R120 94.9 mm to (86.2, -39.8), turned to 90 degrees
- moved LED2 93.5 mm to (91.9, -44.8)
- moved T2 93.5 mm to (90.7, -40.3)
- moved R122 89.3 mm to (95.5, -44.9), turned to 270 degrees
- moved R121 88.4 mm to (95.5, -39.8)
- moved C40 82.8 mm to (29.6, -68.8), turned to 90 degrees
- moved R4 81.1 mm to (14.0, -23.3), turned to 180 degrees
- moved R5 80.1 mm to (14.1, -20.5), turned to 180 degrees
- moved JP30 79.8 mm to (29.2, -74.1), turned to 90 degrees
- moved LED1 78.6 mm to (91.9, -55.2)
- moved T1 78.6 mm to (90.7, -51.1)
- moved R124 76.7 mm to (29.4, -79.6), turned to 0 degrees
- moved C24 76.1 mm to (24.0, 69.8)
- moved C26 76.1 mm to (106.8, 63.4)
- moved C35 76.1 mm to (69.7, 151.9)
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Routing:
- net +3V3: track 6.97 -> 193.7 mm, vias 0 -> 2
- net VDDIO: track 4.24 -> 62.3 mm, vias 0 -> 1
- net TMS_TXD: track 0.00 -> 53.2 mm, vias 0 -> 1
- net USB_VCC: track 5.71 -> 45.3 mm, vias 0 -> 2
- net LED1: track 0.00 -> 31.7 mm, vias 0 -> 2
- net TCK: track 0.00 -> 29.9 mm
- net BUFIN1: track 6.38 -> 34.5 mm, vias 0 -> 2
- net GPIO34: track 4.72 -> 32.2 mm, vias 0 -> 2
- net TDO: track 4.76 -> 28.8 mm
- net TDI: track 0.00 -> 18.7 mm
- net X2CLK: track 11.3 -> 29.1 mm
- net OUT1: track 13.8 -> 29.7 mm, vias 0 -> 1
- net DTR_RESET: track 20.8 -> 5.37 mm, vias 1 -> 0
- net +5V: track 42.7 -> 58.0 mm
- net LIMO1: track 0.00 -> 14.8 mm, vias 0 -> 1
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Other:
- board size 215.6 x 361.3 mm -> 183.2 x 293 mm
