File: March 9/schematic_March8.brd (EAGLE design)
At the start: 183.2 x 293 mm, 314 parts, among them CON1 UBC05V128-B0C04D, IC1 FT232RL, IC10 TL084D, IC13 7805TV, IC3 TL084D, IC4 TL084D, IC5 TL084D, IC6 TL084D, IC7 TL084D, IC8 TL084D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

Commit message: analog routing in progress
Parts:
- moved D13 14.9 mm to (113.1, 66.5)
- moved D15 14.5 mm to (152.3, 66.0)
- moved R25 9.00 mm to (18.6, 162.6)
- moved R20 8.87 mm to (141.4, 75.5)
- moved JP38 8.24 mm to (109.1, 68.9)
- moved R115 7.86 mm to (104.2, 67.0)
- moved R19 7.79 mm to (101.4, 75.8)
- moved R47 7.62 mm to (16.6, 157.3), turned to 90 degrees
- moved C26 7.25 mm to (104.2, 70.1)
- moved JP22 7.04 mm to (136.8, 76.6)
- moved JP21 6.82 mm to (96.7, 77.0)
- moved R114 6.55 mm to (144.2, 66.8)
- moved JP39 6.53 mm to (148.9, 68.0)
- moved R126 6.08 mm to (115.8, 65.8)
- moved R112 6.05 mm to (21.0, 152.2)
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Connections:
- net +5V: no longer R56.1
- net PLS2: now also R56.1
Routing:
- net +5V: track 183.1 -> 220.5 mm, vias 4 -> 8
- net BUFIN3: track 0.00 -> 36.6 mm, vias 0 -> 2
- net BUFIN4: track 0.00 -> 35.4 mm, vias 0 -> 2
- net BUFIN2: track 0.00 -> 35.0 mm, vias 0 -> 2
- net OUT4: track 0.00 -> 31.7 mm, vias 0 -> 1
- net OUT3: track 0.00 -> 30.9 mm, vias 0 -> 1
- net N$20: track 0.00 -> 17.7 mm
- net N$21: track 0.00 -> 17.3 mm
- net N$22: track 0.00 -> 17.0 mm
- net DACO2: track 0.00 -> 13.9 mm
- net LIMO3: track 0.00 -> 13.1 mm, vias 0 -> 1
- net LIMO4: track 0.00 -> 12.8 mm, vias 0 -> 1
- net PLS2: track 0.00 -> 12.2 mm, vias 0 -> 1
- net PLS3: track 0.00 -> 12.0 mm, vias 0 -> 1
- net X3: track 0.00 -> 11.3 mm
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
Commit message: Completed routing of analog part
Parts:
- moved C24 45.8 mm to (21.3, 115.5)
- moved C63 45.8 mm to (33.5, 125.4)
- moved C78 45.8 mm to (20.0, 123.9)
- moved D1 45.8 mm to (29.6, 111.7)
- moved D41 45.8 mm to (36.3, 110.8)
- moved IC3 45.8 mm to (27.4, 124.1)
- moved JP19 45.8 mm to (12.9, 122.5)
- moved JP36 45.8 mm to (26.1, 114.3)
- moved JP46 45.8 mm to (13.5, 129.5)
- moved JP65 45.8 mm to (42.5, 122.8)
- moved R117 45.8 mm to (21.3, 113.1)
- moved R17 45.8 mm to (18.4, 120.7)
- moved R37 45.8 mm to (18.6, 126.1)
- moved R38 45.8 mm to (16.9, 116.4)
- moved R39 45.8 mm to (37.7, 117.8)
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Connections:
- net BUFIN7: now also IC9.12; no longer IC10.12
- net BUFIN8: now also IC10.12; no longer IC9.12
- net LIMO7: now also IC9.13, IC9.14; no longer IC10.13, IC10.14
- net LIMO8: now also IC10.13, IC10.14; no longer IC9.13, IC9.14
Routing:
- net +5V: track 220.5 -> 288.6 mm, vias 8 -> 14
- net OUT7: track 0.00 -> 36.7 mm, vias 0 -> 2
- net OUT8: track 0.00 -> 31.5 mm, vias 0 -> 2
- net OUT5: track 0.00 -> 29.1 mm
- net X7DOT: track 0.00 -> 24.5 mm, vias 0 -> 1
- net BUFIN5: track 0.00 -> 23.8 mm
- net OUT6: track 0.00 -> 21.7 mm
- net BUFIN6: track 0.00 -> 21.5 mm
- net N$55: track 0.00 -> 19.6 mm
- net N$63: track 0.00 -> 19.4 mm
- net LIMO5: track 0.00 -> 19.4 mm, vias 0 -> 1
- net N$62: track 0.00 -> 18.8 mm
- net BUFIN8: track 0.00 -> 18.7 mm
- net N$30: track 0.00 -> 17.4 mm
- net PLS6: track 0.00 -> 16.2 mm, vias 0 -> 1
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