File: March 9/schematic_March8.sch (EAGLE design)
At the start: 314 parts, among them CON1 UBC05V128-B0C04D, IC1 FT232RL, IC10 TL084D, IC13 7805TV, IC3 TL084D, IC4 TL084D, IC5 TL084D, IC6 TL084D, IC7 TL084D, IC8 TL084D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

Commit message: Completed routing of analog part
Connections:
- net BUFIN7: now also IC9D.+IN; no longer IC10D.+IN
- net BUFIN8: now also IC10D.+IN; no longer IC9D.+IN
- net LIMO7: now also IC9D.-IN, IC9D.OUT; no longer IC10D.-IN, IC10D.OUT
- net LIMO8: now also IC10D.-IN, IC10D.OUT; no longer IC9D.-IN, IC9D.OUT
