File: March 10 3.48 pm/schematic_March8.brd (EAGLE design)
At the start: 187.7 x 293.5 mm, 314 parts, among them CON1 UBC05V128-B0C04D, IC1 FT232RL, IC10 TL084D, IC13 7805TV, IC3 TL084D, IC4 TL084D, IC5 TL084D, IC6 TL084D, IC7 TL084D, IC8 TL084D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

Commit message: Done digital (except switches and ADC inputs)
Parts:
- moved JP8 123.8 mm to (115.0, 2.90)
- moved D19 73.0 mm to (115.7, 83.7)
- moved IC10 73.0 mm to (160.0, 92.4)
- moved JP20 73.0 mm to (8.38, 92.6)
- moved JP35 73.0 mm to (158.5, 83.6)
- moved JP39 73.0 mm to (66.1, 84.7)
- moved JP49 73.0 mm to (54.1, 99.6)
- moved JP68 73.0 mm to (82.4, 93.6)
- moved R102 73.0 mm to (166.9, 86.4)
- moved R107 73.0 mm to (152.8, 83.5)
- moved R109 73.0 mm to (105.3, 84.2)
- moved R114 73.0 mm to (61.5, 83.5)
- moved R22 73.0 mm to (15.9, 88.5)
- moved R24 73.0 mm to (61.5, 88.7)
- moved R29 73.0 mm to (20.9, 100.1)
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Connections:
- net N$133: now also U2.5
Routing:
- net USB_VCC: track 45.3 -> 199.1 mm, vias 2 -> 4
- net VDDIO: track 73.2 -> 155.8 mm, vias 1 -> 14
- net GPIO34: track 32.2 -> 109.9 mm, vias 2 -> 4
- net FS: track 1.76 -> 71.0 mm, vias 0 -> 2
- net SPIBMOSI: track 0.00 -> 65.7 mm, vias 0 -> 6
- net TDO: track 28.8 -> 84.3 mm, vias 0 -> 2
- net JTAG_TRST: track 0.00 -> 54.3 mm
- net TMS_RXD: track 4.44 -> 56.6 mm, vias 0 -> 2
- net -5V: track 37.7 -> 76.6 mm
- net +3V3: track 193.7 -> 230.1 mm, vias 2 -> 4
- net SPIBMISO: track 0.00 -> 35.9 mm, vias 0 -> 2
- net SPICLK: track 0.00 -> 34.1 mm, vias 0 -> 2
- net SPIBSS: track 0.00 -> 33.5 mm
- net INTINP1: track 9.89 -> 42.2 mm
- net DACDIN: track 0.00 -> 28.2 mm, vias 0 -> 2
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Other:
- board size 187.7 x 293.5 mm -> 187.3 x 206.7 mm
