File: March 10 4.50 pm/schematic_March8.brd (EAGLE design)
At the start: 187.7 x 293.5 mm, 314 parts, among them CON1 UBC05V128-B0C04D, IC1 FT232RL, IC10 TL084D, IC13 7805TV, IC3 TL084D, IC4 TL084D, IC5 TL084D, IC6 TL084D, IC7 TL084D, IC8 TL084D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

Commit message: Analog internal routing
Parts:
- moved R97 80.7 mm to (125.7, 86.8)
- moved R107 80.7 mm to (125.7, 80.9)
- moved C39 80.7 mm to (125.7, 83.9)
- moved R131 80.1 mm to (137.2, 82.5), turned to 270 degrees
- moved R103 79.4 mm to (136.9, 89.0), turned to 270 degrees
- moved JP72 79.4 mm to (146.6, 93.4)
- moved R109 78.5 mm to (86.6, 81.2)
- moved C35 78.5 mm to (86.6, 83.8)
- moved R79 78.5 mm to (86.6, 86.4)
- moved D22 78.4 mm to (139.9, 82.2), turned to 90 degrees
- moved R129 78.3 mm to (98.3, 82.0)
- moved R90 78.2 mm to (135.6, 100.0)
- moved IC10 78.0 mm to (131.6, 93.1)
- moved R92 78.0 mm to (123.3, 95.8)
- moved C71 78.0 mm to (124.5, 93.1)
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Routing:
- net USB_VCC: track 75.0 -> 199.1 mm, vias 2 -> 4
- net -5V: track 37.7 -> 120.2 mm
- net SPIBMISO: track 0.00 -> 35.9 mm, vias 0 -> 2
- net INTINP4: track 0.00 -> 35.0 mm
- net INTINP7: track 6.25 -> 40.9 mm
- net INTINP8: track 11.9 -> 45.3 mm
- net INTINP1: track 9.89 -> 42.2 mm
- net INTINP2: track 9.86 -> 40.2 mm
- net INTINP3: track 8.72 -> 35.3 mm
- net INTINP5: track 8.44 -> 34.3 mm
- net SWITCH1: track 0.00 -> 23.5 mm
- net SWITCH7: track 0.00 -> 21.8 mm
- net INTINP6: track 13.4 -> 35.0 mm
- net SWITCH2: track 0.00 -> 21.3 mm
- net ADCINA4: track 0.00 -> 19.0 mm
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Other:
- board size 187.7 x 293.5 mm -> 153.4 x 206.1 mm
