File: March 11 Parth's modification/schematic_March8.brd (EAGLE design)
At the start: 180.6 x 197 mm, 314 parts, among them CON1 UBC05V128-B0C04D, IC1 FT232RL, IC10 TL084D, IC13 7805TV, IC3 TL084D, IC4 TL084D, IC5 TL084D, IC6 TL084D, IC7 TL084D, IC8 TL084D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

Commit message: Near Completion
Routing:
- net ADCINA5: track 77.1 -> 146.4 mm, vias 1 -> 2
- net ADCINA2: track 24.1 -> 90.2 mm
- net ADCINA6: track 89.4 -> 39.1 mm
- net ADCINA4: track 73.1 -> 112.2 mm, vias 1 -> 2
- net INTINP1: track 139.9 -> 144.2 mm
- net SWITCH1: track 124.2 -> 126.9 mm
Changed lines of the file:
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@@
 <wire x1="44.32725" y1="-42.2402" x2="45.19205" y2="-41.3754" width="0.254" layer="1"/>
 <wire x1="40.767" y1="-42.2402" x2="44.32725" y2="-42.2402" width="0.254" layer="1"/>
-<wire x1="39.497" y1="-25.0698" x2="32.2326" y2="35.8494875" width="0" layer="19" extent="16-16"/>
+<wire x1="32.2326" y1="36.1188" x2="34.8742" y2="33.4772" width="0.254" layer="16"/>
+<wire x1="34.8742" y1="33.4772" x2="34.8742" y2="-23.749" width="0.254" layer="16"/>
+<wire x1="34.8742" y1="-23.749" x2="36.195" y2="-25.0698" width="0.254" layer="16"/>
+<wire x1="36.195" y1="-25.0698" x2="39.497" y2="-25.0698" width="0.254" layer="16"/>
 </signal>
 <signal name="ADCINB2">
@@
 <contactref element="U1" pad="16"/>
 <contactref element="JP66" pad="2"/>
-<wire x1="67.9704" y1="36.6522" x2="65.7606" y2="34.4424" width="0.254" layer="1"/>
-<wire x1="65.7606" y1="34.4424" x2="65.7606" y2="26.21855" width="0.254" layer="1"/>
 <via x="40.3352" y="-24.9682" extent="1-16" drill="0.254"/>
-<wire x1="40.1828" y1="13.87849375" x2="40.1828" y2="-24.8158" width="0.254" layer="16"/>
+<wire x1="40.1828" y1="13.87849375" x2="40.1828" y2="13.5636" width="0.254" layer="16"/>
+<wire x1="40.1828" y1="13.5636" x2="40.1828" y2="-24.8158" width="0.254" layer="16"/>
 <wire x1="40.1828" y1="-24.8158" x2="40.3352" y2="-24.9682" width="0.254" layer="16"/>
 <wire x1="40.3352" y1="-24.9682" x2="41.3004" y2="-25.9334" width="0.254" layer="1"/>
@@
 <wire x1="45.0940875" y1="-40.8627" x2="46.482" y2="-40.8627" width="0.254" layer="1"/>
 <wire x1="46.482" y1="-40.8627" x2="46.4947" y2="-40.8754" width="0.254" layer="1"/>
-<wire x1="40.1828" y1="13.87849375" x2="65.7606" y2="26.21855" width="0" layer="19" extent="1-16"/>
+<wire x1="67.9704" y1="36.6522" x2="67.9704" y2="36.3828875" width="0.254" layer="1"/>
+<wire x1="67.9704" y1="36.3828875" x2="69.7992" y2="34.5540875" width="0.254" layer="1"/>
+<wire x1="69.7992" y1="34.5540875" x2="69.7992" y2="23.5712" width="0.254" layer="1"/>
+<wire x1="69.7992" y1="23.5712" x2="67.7672" y2="21.5392" width="0.254" layer="1"/>
+<wire x1="67.7672" y1="21.5392" x2="42.672" y2="21.5392" width="0.254" layer="1"/>
+<via x="42.672" y="21.5392" extent="1-16" drill="0.254"/>
+<wire x1="42.672" y1="21.5392" x2="40.1828" y2="19.05" width="0.254" layer="16"/>
+<wire x1="40.1828" y1="19.05" x2="40.1828" y2="13.87849375" width="0.254" layer="16"/>
 </signal>
 <signal name="DACDOUT">
@@
 <wire x1="102.3874" y1="36.5252" x2="102.3874" y2="36.2558875" width="0.254" layer="1"/>
 <wire x1="102.3874" y1="36.2558875" x2="104.2162" y2="34.4270875" width="0.254" layer="1"/>
-<wire x1="104.2162" y1="34.4270875" x2="104.2162" y2="20.8534" width="0.254" layer="1"/>
+<wire x1="104.2162" y1="34.4270875" x2="104.2162" y2="12.2936" width="0.254" layer="1"/>
 <via x="41.275" y="-24.9682" extent="1-16" drill="0.254"/>
-<wire x1="40.9702" y1="13.87743125" x2="40.9702" y2="-24.6634" width="0.254" layer="16"/>
+<wire x1="40.9702" y1="10.4648" x2="40.9702" y2="-24.6634" width="0.254" layer="16"/>
 <wire x1="40.9702" y1="-24.6634" x2="41.275" y2="-24.9682" width="0.254" layer="16"/>
 <wire x1="41.275" y1="-24.9682" x2="41.8084" y2="-25.5016" width="0.254" layer="1"/>
@@
 <wire x1="41.8084" y1="-41.3766" x2="43.969525" y2="-41.3766" width="0.254" layer="1"/>
 <wire x1="43.969525" y1="-41.3766" x2="44.915225" y2="-40.4309" width="0.254" layer="1"/>
-<wire x1="40.9702" y1="13.87743125" x2="104.2162" y2="20.8534" width="0" layer="19" extent="1-16"/>
+<wire x1="104.2162" y1="12.2936" x2="103.378" y2="11.4554" width="0.254" layer="1"/>
+<wire x1="103.378" y1="11.4554" x2="103.2764" y2="11.557" width="0.254" layer="1"/>
+<wire x1="103.2764" y1="11.557" x2="102.997" y2="11.557" width="0.254" layer="1"/>
+<via x="102.997" y="11.557" extent="1-16" drill="0.254"/>
+<wire x1="102.997" y1="11.557" x2="42.0624" y2="11.557" width="0.254" layer="16"/>
+<wire x1="42.0624" y1="11.557" x2="40.9702" y2="10.4648" width="0.254" layer="16"/>
 </signal>
 <signal name="ADCINB4">
@@
 <wire x1="137.7188" y1="37.6020875" x2="139.5476" y2="35.7732875" width="0.254" layer="16"/>
 <wire x1="139.5476" y1="35.7732875" x2="139.5476" y2="27.432" width="0.254" layer="16"/>
-<wire x1="134.3406" y1="22.225" x2="102.4128" y2="22.225" width="0.254" layer="16"/>
-<wire x1="102.4128" y1="22.225" x2="89.4334" y2="9.2456" width="0.254" layer="16"/>
 <wire x1="139.5476" y1="27.432" x2="134.3406" y2="22.225" width="0.254" layer="16"/>
-<wire x1="42.3164" y1="-25.0698" x2="89.4334" y2="9.2456" width="0" layer="19" extent="1-16"/>
+<wire x1="42.3164" y1="-25.0698" x2="134.3406" y2="22.225" width="0" layer="19" extent="1-16"/>
 </signal>
 <signal name="N$41">
@@
 <wire x1="4.2672" y1="30.2764" x2="4.2672" y2="24.4856" width="0.254" layer="1"/>
 <wire x1="4.2672" y1="24.4856" x2="12.065" y2="16.6878" width="0.254" layer="1"/>
-<wire x1="97.1804" y1="-10.1219" x2="94.9706" y2="-12.3317" width="0" layer="19" extent="1-1"/>
+<wire x1="97.1804" y1="-10.1219" x2="96.9899" y2="-10.3124" width="0.254" layer="1"/>
+<wire x1="96.9899" y1="-10.3124" x2="94.9706" y2="-10.3124" width="0.254" layer="1"/>
+<wire x1="94.9706" y1="-10.3124" x2="94.9706" y2="-12.3317" width="0.254" layer="1"/>
 </signal>
 <signal name="INTINP2">
@@
 <wire x1="97.6376" y1="15.3924" x2="95.5294" y2="17.5006" width="0.254" layer="1"/>
 <wire x1="95.5294" y1="17.5006" x2="12.319" y2="17.5006" width="0.254" layer="1"/>
-<wire x1="97.6376" y1="-10.9347" x2="96.2406" y2="-12.3317" width="0" layer="19" extent="1-1"/>
+<wire x1="97.6376" y1="-10.9347" x2="96.4311" y2="-10.9347" width="0.254" layer="1"/>
+<wire x1="96.4311" y1="-10.9347" x2="96.2406" y2="-11.1252" width="0.254" layer="1"/>
+<wire x1="96.2406" y1="-11.1252" x2="96.2406" y2="-12.3317" width="0.254" layer="1"/>
 </signal>
 <signal name="SWITCH2">
