File: March 12 6.43 PM/schematic_March8.sch (EAGLE design)
At the start: 314 parts, among them CON1 UBC05V128-B0C04D, IC1 FT232RL, IC10 TL084D, IC13 7805TV, IC3 TL084D, IC4 TL084D, IC5 TL084D, IC6 TL084D, IC7 TL084D, IC8 TL084D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

Commit message: Brought components closer
Parts:
- D1, D11, D13, D15, D17, D19, D21, D23: value 1SMA5913BT3G -> 1N914BWS; device zener:1SMA5913BT3G -> many_diodes:1N914BWS
Connections:
- net +3V3: now also D1.C, D11.C, D13.C, D15.C, D17.C, D19.C, D21.C, D23.C
- net ADCINA0: now also JP69.2; no longer JP70.2
- net ADCINA1: now also JP70.2; no longer JP69.2
- net ADCINA2: now also JP65.2; no longer JP68.2
- net ADCINA4: now also JP66.2; no longer JP67.2
- net ADCINA5: now also JP67.2; no longer JP66.2
- net ADCINA6: now also JP68.2; no longer JP65.2
- net ADCINB0: now also JP72.2; no longer JP71.2
- net ADCINB1: now also JP71.2; no longer JP72.2
- net AGND: now also C36.2, C42.2, C44.2, C45.2; no longer D1.A, D11.A, D13.A, D15.A, D17.A, D19.A, D21.A, D23.A
- net BUFIN1: now also D1.A; no longer D1.C
- net BUFIN2: now also D11.A; no longer D11.C
- net BUFIN3: now also D13.A; no longer D13.C
- net BUFIN4: now also D15.A; no longer D15.C
- net BUFIN5: now also D17.A; no longer D17.C
- net BUFIN6: now also D19.A; no longer D19.C
- net BUFIN7: now also D21.A; no longer D21.C
- net BUFIN8: now also D23.A; no longer D23.C
- net GND: no longer C36.2, C42.2, C44.2, C45.2
- net INTINP1: now also U9.NO7; no longer U9.NO0
- net INTINP2: now also U9.NO6; no longer U9.NO1
- net INTINP3: now also U9.NO5; no longer U9.NO2
- net INTINP4: now also U9.NO4; no longer U9.NO3
- net INTINP5: now also U9.COM3; no longer U9.NO4
- net INTINP6: now also U9.COM2; no longer U9.NO5
- net INTINP7: now also U9.COM1; no longer U9.NO6
- net INTINP8: now also U9.COM0; no longer U9.NO7
- net INT_CONTROL: now also U1.GPIO2/EPWM2A; no longer U1.GPIO8/EPWM5A/ADCSOCAO
- net N$133: now also U2.!PRE
- net SWITCH1: now also U9.COM7; no longer U9.COM0
- net SWITCH2: now also U9.COM6; no longer U9.COM1
- net SWITCH3: now also U9.COM5; no longer U9.COM2
- net SWITCH4: now also U9.COM4; no longer U9.COM3
- net SWITCH5: now also U9.NO3; no longer U9.COM4
- net SWITCH6: now also U9.NO2; no longer U9.COM5
- net SWITCH7: now also U9.NO1; no longer U9.COM6
- net SWITCH8: now also U9.NO0; no longer U9.COM7
