File: Schematic/March 15 rearranged/schematic_March15 (1).sch (EAGLE design)
At the start: 315 parts, among them CON1 UBC05V128-B0C04D, IC1 FT232RL, IC10 TL084D, IC13 7805TV, IC3 TL084D, IC4 TL084D, IC5 TL084D, IC6 TL084D, IC7 TL084D, IC8 TL084D, IC9 TL084D, Q2 BC557, T1 BC547, T2 BC547, U1 TMS320F28069_PN_80, U10 REF2030AIDDCR, U2 TLV5610_PW_20, U3 REF2030AIDDCR, U4 REF2030AIDDCR, U5 TS12A44514DR, U6 TS12A44514DR, U7 TPS7333QD, U8 REF2030AIDDCR, U9 MAX395CWG+

Commit message: Grounding complete
Parts:
- removed D24: (no value), diode:DIODE-DO214AA
- removed D41: 1N914BWS, many_diodes:1N914BWS
- removed JP55: (no value), pinhead:PINHD-1X3
- removed JP56: (no value), pinhead:PINHD-2X3
- removed L1, L3: BKP1005HS221-T, rcl:L-US0204/5
- added D25: (no value), diode:DIODE-DO214AA
- added JP10, JP9: (no value), pinhead:PINHD-1X3
- added R132, R133: 0, resistor:R-US_R1206
- added R134: 0, rcl:R-US_R1206
- D1, D11, D12, D13, D14, D15, D16, D17, D18, D19, D2, D20, D21, D22, D23: value 1N914BWS -> (none); device many_diodes:1N914BWS -> diode:DIODE-DO214AA
- renumbered JP29 to JP11
Connections:
- net N$133 renamed PREBAR
- removed net N$131: JP55.2, U2.DVDD
- removed net SV1-2: JP14.2
- new net DVDD: JP10.2, U2.DVDD
- net +3V3: now also D12.C, D14.C, D16.C, D18.C, D2.C, D20.C, D22.C, D25.C, JP10.3, JP11.1, JP9.1, R132.1, R133.1; no longer D1.C, D11.C, D13.C, D15.C, D17.C, D19.C, D21.C, D23.C, L1.2, L3.2
- net +5V: now also JP10.1, JP11.3; no longer JP11.1, JP55.1, JP56.1
- net ?????: now also JP9.2; no longer JP56.3
- net AGND: now also D1.A, D11.A, D13.A, D15.A, D17.A, D19.A, D21.A, D23.A, JP14.2, R134.1; no longer D12.A, D14.A, D16.A, D18.A, D2.A, D20.A, D22.A, D41.A
- net BUFIN1: now also D1.C, D25.A; no longer D1.A, D41.C
- net BUFIN2: now also D11.C, D2.A; no longer D11.A, D2.C
- net BUFIN3: now also D12.A, D13.C; no longer D12.C, D13.A
- net BUFIN4: now also D14.A, D15.C; no longer D14.C, D15.A
- net BUFIN5: now also D16.A, D17.C; no longer D16.C, D17.A
- net BUFIN6: now also D18.A, D19.C; no longer D18.C, D19.A
- net BUFIN7: now also D20.A, D21.C; no longer D20.C, D21.A
- net BUFIN8: now also D22.A, D23.C; no longer D22.C, D23.A
- net GND: now also JP9.3, R134.2; no longer JP56.5
- net N$7: now also R133.2; no longer L3.1
- net USB_VCC: no longer JP11.3, JP55.3, JP56.4
- net VDDIO: now also R132.2; no longer L1.1
