File: Schematic/March 16 3.00AM/schematic_March16.brd (EAGLE design)
At the start: 167.3 x 150.8 mm, 314 parts, among them CON1 UBC05V128-B0C04D, IC1 FT232RL, IC10 TL084D, IC13 7805TV, IC3 TL084D, IC4 TL084D, IC5 TL084D, IC6 TL084D, IC7 TL084D, IC8 TL084D, IC9 TL084D, Q2 BC557, T1 BC547, T2 BC547, U1 TMS320F28069_PN_80, U10 REF2030AIDDCR, U2 TLV5610_PW_20, U3 REF2030AIDDCR, U4 REF2030AIDDCR, U5 TS12A44514DR, U6 TS12A44514DR, U7 TPS7333QD, U8 REF2030AIDDCR, U9 MAX395CWG+

Commit message: Grounding complete
Parts:
- added R134: 0, rcl:R1206
- moved C42 12.1 mm to (83.6, -14.6), turned to 270 degrees
- moved R8 3.09 mm to (19.5, -73.7)
- moved C5 2.08 mm to (41.3, -31.1), turned to 0 degrees
- moved R9 0.74 mm to (15.0, -75.7)
- moved JP49 0.57 mm to (115.4, 33.5)
- moved JP60 0.06 mm to (159.9, 3.15)
- turned C29 to 0 degrees
Connections:
- removed net SV1-2: JP14.2
- net AGND: now also JP14.2, R134.1
- net GND: now also R134.2
Routing:
- net AGND: track 5.08 -> 28.0 mm, vias 0 -> 7
- net DACO8: track 125.8 -> 142.2 mm
- net GND: track 8.42 -> 24.7 mm, vias 0 -> 4
- net LDACBAR: track 50.2 -> 40.9 mm
- net VDDIO: track 138.7 -> 131.9 mm, vias 9 -> 10
- net -5V: track 638.4 -> 643.4 mm, vias 12 -> 16
- net INT_CONTROL: track 113.7 -> 118.3 mm, vias 10 -> 12
- net INTINP5: track 69.6 -> 74.2 mm
- net DACO5: track 112.7 -> 116.8 mm
- net +1.5V2: track 51.9 -> 48.5 mm
- net N$12: track 12.3 -> 15.1 mm
- net INTSWITCH2: track 28.8 -> 26.4 mm
- net INTINP1: track 135.8 -> 133.4 mm
- net DACO7: track 146.4 -> 144.0 mm, vias 4 -> 6
- net +3V3: track 585.5 -> 583.2 mm, vias 25 -> 41
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- added copper zone on layer 1, net AGND
- added copper zone on layer 16, net AGND
- added copper zone on layer 1, net GND
- added copper zone on layer 16, net GND
Other:
- board size 167.3 x 150.8 mm -> 179.6 x 161.1 mm
- board text added: "BY PARTHASARATHI KHIRWADKAR, PRANIL JOSHI, SARTHAK CONSUL"
- board text added: "DPAC v2.0"
- board text added: "Digitally Programable Analog Computer"
- board text added: "PROF. MUKUL CHANDORKAR EE344: ELETRONICS DESIGN LAB SPRING, 2019, IIT BOMBAY"

Commit message: added component value and names
Parts:
- C24, C25, C26, C27, C28, C35, C38, C39: value (none) -> 4.7nF
- R100, R102, R104, R29, R31, R32, R34, R36, R39, R41, R42, R49, R51, R53, R55, R56, R58, R60, R62, R64, R66, R68, R70, R75, R77, R80, R82, R87, R89, R91, R93, R98: value (none) -> 33k
- R101, R103, R105, R17, R18, R19, R20, R25, R27, R28, R30, R33, R35, R37, R40, R43, R48, R50, R52, R54, R57, R59, R61, R63, R65, R67, R69, R71, R74, R76, R78, R81, R83, R86, R88, R90, R92, R94, R96, R99: value (none) -> 10k
- R21, R22, R23, R24, R26, R79, R95, R97: value (none) -> 200k
- renumbered IC1 to FT232, IC13 to VREG+5, IC2 to VREG-5, JP10 to DAC-DVDD, JP11 to DAC-PB, JP13 to DAC-IN5, JP14 to XFORMER, JP15 to FF, JP16 to DAC-IN6, JP17 to DAC-IN7, JP18 to DAC-IN8, JP19 to DAC-IN1, JP20 to DAC-IN2, JP21 to DAC-IN3, JP22 to DAC-IN4, JP23 to X-PLS6, JP3 to VDD, JP31 to USB-5, JP34 to X-PLS7, JP35 to X-PLS8, JP36 to X-PLS1, JP37 to X-PLS2, JP38 to X-PLS3, JP39 to X-PLS4, JP4 to VSS, JP42 to X5DOT, JP43 to X6DOT, JP44 to X7DOT, JP45 to X8DOT, JP46 to X1DOT, JP47 to X2DOT, JP48 to X3DOT, JP49 to X4DOT, JP58 to +1.5V1, JP59 to +1.5V2, JP61 to +1.5V3, JP63 to +1.5V4, JP64 to BOOT_JP, JP65 to ADCIN1, JP66 to ADCIN2, JP67 to ADCIN3, JP68 to ADCIN4, JP69 to ADCIN5, JP7 to X-PLS5, JP70 to ADCIN6, JP71 to ADCIN7, JP72 to ADCIN8, JP8 to AGND, JP9 to DAC-MODE, U1 to IC-28069, U10 to VREF4, U2 to DAC, U3 to VREF1, U4 to VREF2, U5 to INTZ1-4, U6 to INTZ5-8, U7 to TPS73333, U8 to VREF3, U9 to MAX

Commit message: name placement done
Parts:
- renumbered JP1 to 3V3_OUT, JP30 to VREF+3V3, JP32 to IN-5V, JP5 to IN+5V, JP6 to VCCIO, TPS73333 to TPS7333

Commit message: Minor corrections in DAC connections, decoupling placed for DAC
Changed lines of the file:
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@@
 <grid distance="1" unitdist="mil" unit="mil" style="dots" multiple="1" display="yes" altdistance="1" altunitdist="mil" altunit="mil"/>
 <layers>
-<layer number="1" name="Top" color="4" fill="1" visible="no" active="yes"/>
+<layer number="1" name="Top" color="4" fill="1" visible="yes" active="yes"/>
 <layer number="2" name="Route2" color="1" fill="3" visible="no" active="no"/>
 <layer number="3" name="Route3" color="4" fill="3" visible="no" active="no"/>
@@
 <layer number="23" name="tOrigins" color="15" fill="1" visible="yes" active="yes"/>
 <layer number="24" name="bOrigins" color="15" fill="1" visible="yes" active="yes"/>
-<layer number="25" name="tNames" color="7" fill="1" visible="no" active="yes"/>
-<layer number="26" name="bNames" color="7" fill="1" visible="no" active="yes"/>
+<layer number="25" name="tNames" color="7" fill="1" visible="yes" active="yes"/>
+<layer number="26" name="bNames" color="7" fill="1" visible="yes" active="yes"/>
 <layer number="27" name="tValues" color="7" fill="1" visible="no" active="yes"/>
 <layer number="28" name="bValues" color="7" fill="1" visible="no" active="yes"/>
@@
 <wire x1="12.5984" y1="-22.5806" x2="13.2842" y2="-22.5806" width="0.2794" layer="16"/>
 <wire x1="56.8614" y1="-44.7421" x2="56.8614" y2="-43.6788" width="0.3048" layer="1"/>
-<wire x1="55.8516" y1="-41.3258" x2="55.9532" y2="-41.4274" width="0.3048" layer="16"/>
 <wire x1="56.4866" y1="-44.323" x2="54.9402" y2="-44.323" width="0.3048" layer="16"/>
 <wire x1="54.9402" y1="-44.323" x2="54.1782" y2="-43.561" width="0.3048" layer="16"/>
@@
 <via x="78.2574" y="-47.1678" extent="1-16" drill="0.254"/>
 <contactref element="R134" pad="2"/>
+<wire x1="8.379" y1="-76.2762" x2="16.7892" y2="-88.3638" width="0" layer="19" extent="1-1"/>
+<wire x1="8.379" y1="-69.6722" x2="8.379" y2="-76.2762" width="0" layer="19" extent="1-1"/>
+<wire x1="8.379" y1="-65.9892" x2="8.379" y2="-69.6722" width="0" layer="19" extent="1-1"/>
+<wire x1="16.3686" y1="-53.7392" x2="8.379" y2="-65.9892" width="0" layer="19" extent="1-1"/>
+<wire x1="18.3186" y1="-53.7392" x2="16.3686" y2="-53.7392" width="0" layer="19" extent="1-1"/>
+<wire x1="20.9186" y1="-53.7392" x2="18.3186" y2="-53.7392" width="0" layer="19" extent="1-1"/>
+<wire x1="18.9686" y1="-46.4892" x2="18.3186" y2="-53.7392" width="0" layer="19" extent="1-1"/>
+<wire x1="30.5562" y1="-54.7116" x2="21.5686" y2="-53.7392" width="0" layer="19" extent="1-1"/>
+<wire x1="28.2448" y1="-42.9768" x2="18.9686" y2="-46.4892" width="0" layer="19" extent="1-1"/>
+<wire x1="36.192" y1="-39.3446" x2="28.2448" y2="-42.9768" width="0" layer="19" extent="16-16"/>
+<wire x1="38.7066" y1="-42.926" x2="36.192" y2="-39.3446" width="0" layer="19" extent="16-16"/>
+<wire x1="34.6964" y1="-33.6804" x2="36.192" y2="-39.3446" width="0" layer="19" extent="16-16"/>
+<wire x1="39.9004" y1="-31.1404" x2="34.6964" y2="-33.6804" width="0" layer="19" extent="16-16"/>
+<wire x1="28.9048" y1="-31.0896" x2="34.6964" y2="-33.6804" width="0" layer="19" extent="1-1"/>
+<wire x1="28.9048" y1="-28.6004" x2="28.9048" y2="-31.0896" width="0" layer="19" extent="1-1"/>
+<wire x1="28.9048" y1="-26.162" x2="28.9048" y2="-28.6004" width="0" layer="19" extent="1-1"/>
+<wire x1="46.4947" y1="-34.3754" x2="39.9004" y2="-31.1404" width="0" layer="19" extent="1-16"/>
+<wire x1="49.7362" y1="-35.2298" x2="46.4947" y2="-34.3754" width="0" layer="19" extent="1-16"/>
+<wire x1="49.914" y1="-31.9786" x2="49.7362" y2="-35.2298" width="0" layer="19" extent="16-16"/>
+<wire x1="51.8614" y1="-31.5087" x2="49.914" y2="-31.9786" width="0" layer="19" extent="1-16"/>
+<wire x1="52.8614" y1="-31.5087" x2="51.8614" y2="-31.5087" width="0" layer="19" extent="1-1"/>
+<wire x1="56.3614" y1="-31.5087" x2="52.8614" y2="-31.5087" width="0" layer="19" extent="1-1"/>
+<wire x1="59.2358" y1="-32.131" x2="56.3614" y2="-31.5087" width="0" layer="19" extent="1-16"/>
+<wire x1="59.2612" y1="-34.8742" x2="59.2358" y2="-32.131" width="0" layer="19" extent="16-16"/>
+<wire x1="59.7281" y1="-38.3754" x2="59.2612" y2="-34.8742" width="0" layer="19" extent="1-16"/>
+<wire x1="53.1114" y1="-36.452" x2="49.7362" y2="-35.2298" width="0" layer="19" extent="16-16"/>
+<wire x1="55.9532" y1="-38.5318" x2="53.1114" y2="-36.452" width="0" layer="19" extent="16-16"/>
+<wire x1="55.9024" y1="-41.3766" x2="55.9532" y2="-38.5318" width="0" layer="19" extent="16-16"/>
+<wire x1="55.9532" y1="-41.4274" x2="55.9024" y2="-41.3766" width="0" layer="19" extent="16-16"/>
+<wire x1="56.8614" y1="-44.7421" x2="56.4866" y2="-44.323" width="0" layer="19" extent="1-16"/>
+<wire x1="51.8614" y1="-44.7421" x2="54.1782" y2="-43.561" width="0" layer="19" extent="1-16"/>
+<wire x1="48.3614" y1="-44.7421" x2="51.8614" y2="-44.7421" width="0" layer="19" extent="1-1"/>
+<wire x1="46.9108" y1="-44.3738" x2="48.3614" y2="-44.7421" width="0" layer="19" extent="1-16"/>
+<wire x1="46.8346" y1="-41.8592" x2="46.9108" y2="-44.3738" width="0" layer="19" extent="16-16"/>
+<wire x1="46.4947" y1="-39.3754" x2="46.8346" y2="-41.8592" width="0" layer="19" extent="1-16"/>
+<wire x1="46.8346" y1="-39.2176" x2="46.4947" y2="-39.3754" width="0" layer="19" extent="1-16"/>
+<wire x1="54.3052" y1="-20.6796" x2="52.8614" y2="-31.5087" width="0" layer="19" extent="1-1"/>
+<wire x1="36.0934" y1="-17.2212" x2="28.9048" y2="-26.162" width="0" layer="19" extent="1-1"/>
+<wire x1="12.8748" y1="-34.3662" x2="18.9686" y2="-46.4892" width="0" layer="19" extent="1-1"/>
+<wire x1="11.2776" y1="-30.4292" x2="12.8748" y2="-34.3662" width="0" layer="19" extent="1-1"/>
+<wire x1="38.4586" y1="-66.2432" x2="30.5562" y2="-54.7116" width="0" layer="19" extent="1-1"/>
+<wire x1="39.2938" y1="-71.5264" x2="38.4586" y2="-66.2432" width="0" layer="19" extent="1-1"/>
+<wire x1="73.9394" y1="-28.4988" x2="59.2358" y2="-32.131" width="0" layer="19" extent="16-16"/>
+<wire x1="79.0194" y1="-28.4988" x2="73.9394" y2="-28.4988" width="0" layer="19" extent="1-1"/>
+<wire x1="81.5594" y1="-28.4988" x2="79.0194" y2="-28.4988" width="0" layer="19" extent="1-1"/>
+<wire x1="84.0994" y1="-28.4988" x2="81.5594" y2="-28.4988" width="0" layer="19" extent="1-1"/>
+<wire x1="73.9902" y1="-18.821" x2="73.9394" y2="-28.4988" width="0" layer="19" extent="1-1"/>
+<wire x1="93.7006" y1="-21.7043" x2="84.0994" y2="-28.4988" width="0" layer="19" extent="1-1"/>
+<wire x1="83.7722" y1="-41.6052" x2="84.0994" y2="-28.4988" width="0" layer="19" extent="16-16"/>
+<wire x1="83.7976" y1="-43.8658" x2="83.7722" y2="-41.6052" width="0" layer="19" extent="16-16"/>
+<wire x1="78.2574" y1="-47.1678" x2="83.7976" y2="-43.8658" width="0" layer="19" extent="16-16"/>
+<wire x1="95.4786" y1="-43.5106" x2="83.7976" y2="-43.8658" width="0" layer="19" extent="1-16"/>
+<wire x1="95.504" y1="-41.173" x2="95.4786" y2="-43.5106" width="0" layer="19" extent="1-1"/>
+<wire x1="95.4786" y1="-51.5362" x2="95.4786" y2="-43.5106" width="0" layer="19" extent="1-1"/>
+<wire x1="95.4786" y1="-53.8484" x2="95.4786" y2="-51.5362" width="0" layer="19" extent="1-1"/>
+<wire x1="99.797" y1="-53.8226" x2="95.4786" y2="-53.8484" width="0" layer="19" extent="1-1"/>
 </signal>
 <signal name="+3V3">
