File: Schematic/March 17 10.39PM/schematic_March16.sch (EAGLE design)
At the start: 317 parts, among them CON1 UBC05V128-B0C04D, IC10 TL084D, IC3 TL084D, IC4 TL084D, IC5 TL084D, IC6 TL084D, IC7 TL084D, IC8 TL084D, IC9 TL084D, Q2 BC557, T1 BC547, T2 BC547, X7DOT Int_inp

Commit message: Made corrections, added RC values
Parts:
- C1, C2: value 36p -> 36pF
- C20, C36, C41, C42, C43, C44, C45, C63, C64, C65, C66, C67, C68, C69, C70, C71, C72, C73, C74, C75, C76, C77, C78, C93, C94, C95: value 2.2u -> 0.1uF
- C29, C3: value 0.1u -> 0.1uF
- C46, C47: value 1uF -> 0.1uF
- R107, R108, R109, R112, R114, R115, R116, R117: value (none) -> 50
- R110, R111: value 1K -> 1k
- R124: value 1 -> 250k
- R125, R126, R127, R128, R129, R130, R131, R14: value (none) -> 1k
- R17, R18, R19, R20, R25, R78, R94, R96: value 10k -> 56k
- R21, R22, R23, R24, R26, R79, R95, R97: value 200k -> 680k
- R38, R44, R45, R46, R47, R73, R84, R85: value (none) -> 12k
- R8, R9: value 33 -> 0
- X-PLS7: value pls -> (none)
- X7DOT: value Int_inp -> (none)
Other:
- moved on the sheet: C37
